Commit message: test passed

File: urdf/uav300_head.urdf (robot description, URDF)
Before this commit: robot uav300_head, 9 links, 8 joints
Joints:
- joint head_joint: axis 0 0 0 -> 0 0 1

Commit message: add view field

File: urdf/uav300_head.urdf (robot description, URDF)
Before this commit: robot uav300_head, 9 links, 8 joints
Links:
- added link view_link, mass 0.399880166519623; collision mesh filename=package://uav300_head/meshes/view_field.stl scale=1 1 1; visual mesh filename=package://uav300_head/meshes/view_field.stl scale=1 1 1
Joints:
- added joint view_joint: type fixed, parent head_link, child view_link, origin xyz=0 0 0 rpy=0 0 0, axis 0 0 1

Commit message: v1.0

File: urdf/uav300_head.urdf (robot description, URDF)
Before this commit: robot uav300_head, 10 links, 9 joints
Links:
- removed link ardrone3_link
- removed link robot1_link
- removed link robot2_link
- removed link robot3_link
- added link ardrone0_link, mass 0.399880166519623; collision mesh filename=package://uav300_head/meshes/Drone_2.0_Complete_Indoor_02.S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 scale=0.001 0.001 0.001; visual mesh filename=package://uav300_head/meshes/Drone_2.0_Complete_Indoor_02.S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 scale=0.001 0.001 0.001
- added link person0_link, mass 0.399880166519623; collision mesh filename=package://uav300_head/meshes/robot.stl scale=0.001 0.001 0.001; visual mesh filename=package://uav300_head/meshes/robot.stl scale=0.001 0.001 0.001
- added link person1_link, mass 0.399880166519623; collision mesh filename=package://uav300_head/meshes/robot.stl scale=0.001 0.001 0.001; visual mesh filename=package://uav300_head/meshes/robot.stl scale=0.001 0.001 0.001
- added link person2_link, mass 0.399880166519623; collision mesh filename=package://uav300_head/meshes/robot.stl scale=0.001 0.001 0.001; visual mesh filename=package://uav300_head/meshes/robot.stl scale=0.001 0.001 0.001
Joints:
- removed joint ardrone3_joint
- removed joint robot1_joint
- removed joint robot2_joint
- removed joint robot3_joint
- added joint ardrone0_joint: type fixed, parent world, child ardrone0_link, origin xyz=1000 1000 0 rpy=0 0 0, axis 0 0 0
- added joint person0_joint: type fixed, parent world, child person0_link, origin xyz=1000 1000 0 rpy=0 0 0, axis 0 0 0
- added joint person1_joint: type fixed, parent world, child person1_link, origin xyz=1000 1000 0 rpy=0 0 0, axis 0 0 0
- added joint person2_joint: type fixed, parent world, child person2_link, origin xyz=1000 1000 0 rpy=0 0 0, axis 0 0 0

Commit message: final

File: urdf/uav300_head.urdf (robot description, URDF)
Before this commit: robot uav300_head, 10 links, 9 joints
Links:
- removed link ardrone0_link
- removed link ardrone1_link
- removed link ardrone2_link
- removed link person0_link
- removed link person1_link
- removed link person2_link
- added link drone0_link, mass 0.399880166519623; collision mesh filename=package://uav300_head/meshes/Drone_2.0_Complete_Indoor_02.S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 scale=0.001 0.001 0.001; visual mesh filename=package://uav300_head/meshes/Drone_2.0_Complete_Indoor_02.S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 scale=0.001 0.001 0.001
- added link drone1_link, mass 0.399880166519623; collision mesh filename=package://uav300_head/meshes/Drone_2.0_Complete_Indoor_02.S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 scale=0.001 0.001 0.001; visual mesh filename=package://uav300_head/meshes/Drone_2.0_Complete_Indoor_02.S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 scale=0.001 0.001 0.001
- added link drone2_link, mass 0.399880166519623; collision mesh filename=package://uav300_head/meshes/Drone_2.0_Complete_Indoor_02.S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 scale=0.001 0.001 0.001; visual mesh filename=package://uav300_head/meshes/Drone_2.0_Complete_Indoor_02.S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 scale=0.001 0.001 0.001
- added link robot0_link, mass 0.399880166519623; collision mesh filename=package://uav300_head/meshes/robot.stl scale=0.001 0.001 0.001; visual mesh filename=package://uav300_head/meshes/robot.stl scale=0.001 0.001 0.001
- added link robot1_link, mass 0.399880166519623; collision mesh filename=package://uav300_head/meshes/robot.stl scale=0.001 0.001 0.001; visual mesh filename=package://uav300_head/meshes/robot.stl scale=0.001 0.001 0.001
- added link robot2_link, mass 0.399880166519623; collision mesh filename=package://uav300_head/meshes/robot.stl scale=0.001 0.001 0.001; visual mesh filename=package://uav300_head/meshes/robot.stl scale=0.001 0.001 0.001
Joints:
- removed joint ardrone0_joint
- removed joint ardrone1_joint
- removed joint ardrone2_joint
- removed joint person0_joint
- removed joint person1_joint
- removed joint person2_joint
- added joint drone0_joint: type fixed, parent world, child drone0_link, origin xyz=1000 1000 0 rpy=0 0 0, axis 0 0 0
- added joint drone1_joint: type fixed, parent world, child drone1_link, origin xyz=1000 1000 0 rpy=0 0 0, axis 0 0 0
- added joint drone2_joint: type fixed, parent world, child drone2_link, origin xyz=1000 1000 0 rpy=0 0 0, axis 0 0 0
- added joint robot0_joint: type fixed, parent world, child robot0_link, origin xyz=1000 1000 0 rpy=0 0 0, axis 0 0 0
- added joint robot1_joint: type fixed, parent world, child robot1_link, origin xyz=1000 1000 0 rpy=0 0 0, axis 0 0 0
- added joint robot2_joint: type fixed, parent world, child robot2_link, origin xyz=1000 1000 0 rpy=0 0 0, axis 0 0 0
